File: pcb/led.kicad_sch (KiCad schematic)
At the start: 3 parts, among them U9 LP5810ADSDR

Commit message: pcb: simplify power supply and define LC filter
Parts:
- D1: symbol Device:LED_BGAR -> Device:LED_GBAR
Connections:
- net at D1.1 (GK): now also U9.7 (OUT1); no longer U9.6 (OUT2)
- net at D1.2 (BK): now also U9.8 (OUT0); no longer U9.7 (OUT1)
- net at D1.4 (RK): now also U9.6 (OUT2); no longer U9.8 (OUT0)
- no-connect marks 0 -> 1
Changed lines of the file:
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@@
 		(color 0 0 0 0)
+	)
+	(no_connect
+		(at 140.97 107.95)
 	)
 	(bus_entry
@@
 	(wire
 		(pts
-			(xy 140.97 92.71) (xy 156.21 92.71)
+			(xy 143.51 102.87) (xy 140.97 102.87)
+		)
+		(stroke
+			(width 0)
+			(type default)
+		)
+	)
+	(wire
+		(pts
+			(xy 153.67 92.71) (xy 156.21 92.71)
+		)
+		(stroke
+			(width 0)
+			(type default)
+		)
+	)
+	(wire
+		(pts
+			(xy 143.51 100.33) (xy 153.67 100.33)
 		)
 		(stroke
@@
 	(wire
 		(pts
-			(xy 140.97 102.87) (xy 156.21 102.87)
-		)
-		(stroke
-			(width 0)
-			(type default)
-		)
-	)
-	(wire
-		(pts
 			(xy 128.27 113.03) (xy 115.57 113.03)
 		)
@@
 	(wire
 		(pts
+			(xy 140.97 92.71) (xy 148.59 92.71)
+		)
+		(stroke
+			(width 0)
+			(type default)
+		)
+	)
+	(wire
+		(pts
 			(xy 177.8 73.66) (xy 177.8 97.79)
 		)
@@
 	(wire
 		(pts
+			(xy 148.59 92.71) (xy 148.59 102.87)
+		)
+		(stroke
+			(width 0)
+			(type default)
+		)
+	)
+	(wire
+		(pts
+			(xy 153.67 100.33) (xy 153.67 92.71)
+		)
+		(stroke
+			(width 0)
+			(type default)
+		)
+	)
+	(wire
+		(pts
 			(xy 128.27 73.66) (xy 177.8 73.66)
 		)
@@
 	(wire
 		(pts
+			(xy 143.51 102.87) (xy 143.51 100.33)
+		)
+		(stroke
+			(width 0)
+			(type default)
+		)
+	)
+	(wire
+		(pts
 			(xy 140.97 97.79) (xy 156.21 97.79)
 		)
@@
 		(pts
 			(xy 107.95 73.66) (xy 116.84 73.66)
+		)
+		(stroke
+			(width 0)
+			(type default)
+		)
+	)
+	(wire
+		(pts
+			(xy 148.59 102.87) (xy 156.21 102.87)
 		)
 		(stroke
@@
 	)
 	(symbol
-		(lib_id "Device:LED_BGAR")
+		(lib_id "Device:LED_GBAR")
 		(at 161.29 97.79 0)
 		(unit 1)
@@
 			)
 		)
-		(property "Description" "RGB LED, blue/green/anode/red"
+		(property "Description" "RGB LED, green/blue/anode/red"
 			(at 161.29 97.79 0)
 			(effects

Commit message: pcb: pretty much the final version
Parts:
- C37: manf# (none) -> CL10B105KP8NNNC
- D1: manf# (none) -> QBLP615-RGB-3053
- U9: manf# (none) -> LP5810ADSDR
Changed lines of the file:
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@@
+			)
+		)
+		(property "manf#" "QBLP615-RGB-3053"
+			(at 161.29 97.79 0)
+			(effects
+				(font
+					(size 1.27 1.27)
+				)
+				(hide yes)
 			)
 		)
@@
 			)
 		)
+		(property "manf#" "LP5810ADSDR"
+			(at 128.27 100.33 0)
+			(effects
+				(font
+					(size 1.27 1.27)
+				)
+				(hide yes)
+			)
+		)
 		(pin "8"
 		)
@@
 			)
 		)
-		(property "Description" "Decoupling"
+		(property "Description" "Capacitor, decoupling, 10V, X7R"
 			(at 116.84 77.47 0)
 			(effects
+				(font
+					(size 1.27 1.27)
+				)
+				(hide yes)
+			)
+		)
+		(property "manf#" "CL10B105KP8NNNC"
+			(at 116.84 77.47 0)
+			(effects
